Commit message: Work on launch files, add xyz args to spawn_statek.launch

File: catkin_ws/src/statek_rviz/urdf/statek.urdf (robot description, URDF)
Before this commit: robot statek, 1 links, 0 joints
Links:
- removed link base_link
- added link $(arg statek_name)_base_link; visual mesh filename=file://$(find statek_rviz)/urdf/chassis.dae
