Commit message: Merge statek_description into statek_config, add dynamic transform publisher node draft, optimize statek motor plugin and model physics in Gazebo, rename ds4 teleop node in statek_teleop

File: catkin_ws/src/statek_config/urdf/statek.urdf (robot description, URDF)
Before this commit: robot statek, 5 links, 4 joints
Links:
- link $(arg statek_name)/base_link: geometry collision box size=.62 .9 .15; visual mesh filename=file://$(find statek_config)/urdf/chassis.dae scale=1.0 1.0 1.0
- link $(arg statek_name)/left_back_wheel: geometry collision sphere length=0.07 radius=0.12; visual mesh filename=file://$(find statek_config)/urdf/wheel.dae scale=1.0 1.0 1.0
- link $(arg statek_name)/left_front_wheel: geometry collision sphere length=0.07 radius=0.12; visual mesh filename=file://$(find statek_config)/urdf/wheel.dae scale=1.0 1.0 1.0
- link $(arg statek_name)/right_back_wheel: geometry collision sphere length=0.07 radius=0.12; visual mesh filename=file://$(find statek_config)/urdf/wheel.dae scale=1.0 1.0 1.0
- link $(arg statek_name)/right_front_wheel: geometry collision sphere length=0.07 radius=0.12; visual mesh filename=file://$(find statek_config)/urdf/wheel.dae scale=1.0 1.0 1.0

Commit message: Add Encoder message, fix .gitignore to include ros package.xml files, cleanup package.xml and CMakeLists.txt

File: catkin_ws/src/statek_config/urdf/statek.urdf (robot description, URDF)
Before this commit: robot statek, 5 links, 4 joints
Links:
- link $(arg statek_name)/base_link: mass 14 -> 9

Commit message: Add encoder publishers, fix URDF links and joints, add code to dynamic transform publisher

File: catkin_ws/src/statek_config/urdf/statek.urdf (robot description, URDF)
Before this commit: robot statek, 5 links, 4 joints
Links:
- removed link $(arg statek_name)/left_back_wheel
- removed link $(arg statek_name)/left_front_wheel
- removed link $(arg statek_name)/right_back_wheel
- removed link $(arg statek_name)/right_front_wheel
- added link $(arg statek_name)/left_back_wheel_link, mass 1.3; collision sphere length=0.07 radius=0.12; visual mesh filename=file://$(find statek_config)/urdf/wheel.dae scale=1.0 1.0 1.0
- added link $(arg statek_name)/left_front_wheel_link, mass 1.3; collision sphere length=0.07 radius=0.12; visual mesh filename=file://$(find statek_config)/urdf/wheel.dae scale=1.0 1.0 1.0
- added link $(arg statek_name)/right_back_wheel_link, mass 1.3; collision sphere length=0.07 radius=0.12; visual mesh filename=file://$(find statek_config)/urdf/wheel.dae scale=1.0 1.0 1.0
- added link $(arg statek_name)/right_front_wheel_link, mass 1.3; collision sphere length=0.07 radius=0.12; visual mesh filename=file://$(find statek_config)/urdf/wheel.dae scale=1.0 1.0 1.0
Joints:
- joint left_back_wheel_hinge: child $(arg statek_name)/left_back_wheel -> $(arg statek_name)/left_back_wheel_link; origin xyz=-0.252682 0.270467 -0.03126 rpy=0      0     -1.5708 -> xyz=-0.252682 0.270467 -0.03126 rpy=0      0     1.5708
- joint left_front_wheel_hinge: child $(arg statek_name)/left_front_wheel -> $(arg statek_name)/left_front_wheel_link; origin xyz=0.167807 0.270467 -0.03126 rpy=0      0     -1.5708 -> xyz=0.167807 0.270467 -0.03126 rpy=0      0     1.5708
- joint right_back_wheel_hinge: child $(arg statek_name)/right_back_wheel -> $(arg statek_name)/right_back_wheel_link
- joint right_front_wheel_hinge: child $(arg statek_name)/right_front_wheel -> $(arg statek_name)/right_front_wheel_link

Commit message: Add multiple cameras to Gazebo

File: catkin_ws/src/statek_config/urdf/statek.urdf (robot description, URDF)
Before this commit: robot statek, 5 links, 4 joints
Links:
- removed link $(arg statek_name)/left_back_wheel_link
- removed link $(arg statek_name)/left_front_wheel_link
- removed link $(arg statek_name)/right_back_wheel_link
- removed link $(arg statek_name)/right_front_wheel_link
- added link $(arg statek_name)/wheels/left_back_link, mass 1.3; collision sphere length=0.07 radius=0.12; visual mesh filename=file://$(find statek_config)/urdf/wheel.dae scale=1.0 1.0 1.0
- added link $(arg statek_name)/wheels/left_front_link, mass 1.3; collision sphere length=0.07 radius=0.12; visual mesh filename=file://$(find statek_config)/urdf/wheel.dae scale=1.0 1.0 1.0
- added link $(arg statek_name)/wheels/right_back_link, mass 1.3; collision sphere length=0.07 radius=0.12; visual mesh filename=file://$(find statek_config)/urdf/wheel.dae scale=1.0 1.0 1.0
- added link $(arg statek_name)/wheels/right_front_link, mass 1.3; collision sphere length=0.07 radius=0.12; visual mesh filename=file://$(find statek_config)/urdf/wheel.dae scale=1.0 1.0 1.0
Joints:
- joint left_back_wheel_hinge: child $(arg statek_name)/left_back_wheel_link -> $(arg statek_name)/wheels/left_back_link
- joint left_front_wheel_hinge: child $(arg statek_name)/left_front_wheel_link -> $(arg statek_name)/wheels/left_front_link
- joint right_back_wheel_hinge: child $(arg statek_name)/right_back_wheel_link -> $(arg statek_name)/wheels/right_back_link
- joint right_front_wheel_hinge: child $(arg statek_name)/right_front_wheel_link -> $(arg statek_name)/wheels/right_front_link
