Commit message: Add park map, force rviz markers to be visible until next update, work a bit with Gazebo urdf model

File: catkin_ws/src/statek_config/urdf/robot_description.urdf (robot description, URDF)
Before this commit: robot statek, 5 links, 4 joints
Links:
- link $(arg statek_name)/base_link: geometry collision box size=0.62 0.9 0.15; visual mesh filename=file://$(find statek_config)/urdf/chassis.dae scale=1.0 1.0 1.0
Joints:
- joint left_back_wheel_hinge: axis 1  0  0 -> 1 0 0; origin xyz=-0.252682 0.270467 -0.03126 rpy=0      0     1.5708 -> xyz=-0.252682 0.270467 -0.03126 rpy=0 0 1.5708
- joint left_front_wheel_hinge: axis 1  0  0 -> 1 0 0; origin xyz=0.167807 0.270467 -0.03126 rpy=0      0     1.5708 -> xyz=0.167807 0.270467 -0.03126 rpy=0 0 1.5708
- joint right_back_wheel_hinge: axis 1  0  0 -> 1 0 0; origin xyz=-0.252682 -0.264541 -0.03126 rpy=0      0      1.5708 -> xyz=-0.252682 -0.264541 -0.03126 rpy=0 0 1.5708
- joint right_front_wheel_hinge: axis 1  0  0 -> 1 0 0; origin xyz=0.167807 -0.264541 -0.03126 rpy=0      0      1.5708 -> xyz=0.167807 -0.264541 -0.03126 rpy=0 0 1.5708
