File: electronics/button_panel/button_panel.sch (KiCad schematic (older format))
At the start: 31 parts, among them J1 Conn_01x10, J2 Conn_01x09, SW1 PWR, SW2 RST, SW3 AP, SW4 MAN, SW5 FC REC, SW6 USR1, SW7 USR2, SW8 USR3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

Commit message: Edit button panel, edit CAD, add motor tensioners
Parts:
- R1, R10, R11, R12, R13, R2, R3, R4, R5, R6, R7, R8, R9: footprint Resistor_THT:R_Axial_DIN0309_L9.0mm_D3.2mm_P12.70mm_Horizontal -> Resistor_SMD:R_1206_3216Metric_Pad1.42x1.75mm_HandSolder
Changed lines of the file:
@@
 F 0 "R4" H 4750 3650 50  0000 L CNN
 F 1 "R" H 4800 3550 50  0000 L CNN
-F 2 "Resistor_THT:R_Axial_DIN0309_L9.0mm_D3.2mm_P12.70mm_Horizontal" V 4880 3600 50  0001 C CNN
+F 2 "Resistor_SMD:R_1206_3216Metric_Pad1.42x1.75mm_HandSolder" V 4880 3600 50  0001 C CNN
 F 3 "~" H 4950 3600 50  0001 C CNN
 	1    4950 3600
@@
 F 0 "R3" H 4670 3646 50  0000 L CNN
 F 1 "R" H 4670 3555 50  0000 L CNN
-F 2 "Resistor_THT:R_Axial_DIN0309_L9.0mm_D3.2mm_P12.70mm_Horizontal" V 4530 3600 50  0001 C CNN
+F 2 "Resistor_SMD:R_1206_3216Metric_Pad1.42x1.75mm_HandSolder" V 4530 3600 50  0001 C CNN
 F 3 "~" H 4600 3600 50  0001 C CNN
 	1    4600 3600
@@
 F 0 "R2" H 4370 3646 50  0000 L CNN
 F 1 "R" H 4370 3555 50  0000 L CNN
-F 2 "Resistor_THT:R_Axial_DIN0309_L9.0mm_D3.2mm_P12.70mm_Horizontal" V 4230 3600 50  0001 C CNN
+F 2 "Resistor_SMD:R_1206_3216Metric_Pad1.42x1.75mm_HandSolder" V 4230 3600 50  0001 C CNN
 F 3 "~" H 4300 3600 50  0001 C CNN
 	1    4300 3600
@@
 F 0 "R6" H 7970 3246 50  0000 L CNN
 F 1 "R" H 7970 3155 50  0000 L CNN
-F 2 "Resistor_THT:R_Axial_DIN0309_L9.0mm_D3.2mm_P12.70mm_Horizontal" V 7830 3200 50  0001 C CNN
+F 2 "Resistor_SMD:R_1206_3216Metric_Pad1.42x1.75mm_HandSolder" V 7830 3200 50  0001 C CNN
 F 3 "~" H 7900 3200 50  0001 C CNN
 	1    7900 3200
@@
 F 0 "R5" H 7970 2696 50  0000 L CNN
 F 1 "R" H 7970 2605 50  0000 L CNN
-F 2 "Resistor_THT:R_Axial_DIN0309_L9.0mm_D3.2mm_P12.70mm_Horizontal" V 7830 2650 50  0001 C CNN
+F 2 "Resistor_SMD:R_1206_3216Metric_Pad1.42x1.75mm_HandSolder" V 7830 2650 50  0001 C CNN
 F 3 "~" H 7900 2650 50  0001 C CNN
 	1    7900 2650
@@
 F 0 "R9" H 3970 3646 50  0000 L CNN
 F 1 "R" H 3970 3555 50  0000 L CNN
-F 2 "Resistor_THT:R_Axial_DIN0309_L9.0mm_D3.2mm_P12.70mm_Horizontal" V 3830 3600 50  0001 C CNN
+F 2 "Resistor_SMD:R_1206_3216Metric_Pad1.42x1.75mm_HandSolder" V 3830 3600 50  0001 C CNN
 F 3 "~" H 3900 3600 50  0001 C CNN
 	1    3900 3600
@@
 F 0 "R8" H 3570 3646 50  0000 L CNN
 F 1 "R" H 3570 3555 50  0000 L CNN
-F 2 "Resistor_THT:R_Axial_DIN0309_L9.0mm_D3.2mm_P12.70mm_Horizontal" V 3430 3600 50  0001 C CNN
+F 2 "Resistor_SMD:R_1206_3216Metric_Pad1.42x1.75mm_HandSolder" V 3430 3600 50  0001 C CNN
 F 3 "~" H 3500 3600 50  0001 C CNN
 	1    3500 3600
@@
 F 0 "R7" H 3170 3646 50  0000 L CNN
 F 1 "R" H 3170 3555 50  0000 L CNN
-F 2 "Resistor_THT:R_Axial_DIN0309_L9.0mm_D3.2mm_P12.70mm_Horizontal" V 3030 3600 50  0001 C CNN
+F 2 "Resistor_SMD:R_1206_3216Metric_Pad1.42x1.75mm_HandSolder" V 3030 3600 50  0001 C CNN
 F 3 "~" H 3100 3600 50  0001 C CNN
 	1    3100 3600
@@
 F 0 "R1" H 2770 3646 50  0000 L CNN
 F 1 "R" H 2770 3555 50  0000 L CNN
-F 2 "Resistor_THT:R_Axial_DIN0309_L9.0mm_D3.2mm_P12.70mm_Horizontal" V 2630 3600 50  0001 C CNN
+F 2 "Resistor_SMD:R_1206_3216Metric_Pad1.42x1.75mm_HandSolder" V 2630 3600 50  0001 C CNN
 F 3 "~" H 2700 3600 50  0001 C CNN
 	1    2700 3600
@@
 F 0 "R10" H 6320 5346 50  0000 L CNN
 F 1 "R" H 6320 5255 50  0000 L CNN
-F 2 "Resistor_THT:R_Axial_DIN0309_L9.0mm_D3.2mm_P12.70mm_Horizontal" V 6180 5300 50  0001 C CNN
+F 2 "Resistor_SMD:R_1206_3216Metric_Pad1.42x1.75mm_HandSolder" V 6180 5300 50  0001 C CNN
 F 3 "~" H 6250 5300 50  0001 C CNN
 	1    6250 5300
@@
 F 0 "R11" H 6520 4896 50  0000 L CNN
 F 1 "R" H 6520 4805 50  0000 L CNN
-F 2 "Resistor_THT:R_Axial_DIN0309_L9.0mm_D3.2mm_P12.70mm_Horizontal" V 6380 4850 50  0001 C CNN
+F 2 "Resistor_SMD:R_1206_3216Metric_Pad1.42x1.75mm_HandSolder" V 6380 4850 50  0001 C CNN
 F 3 "~" H 6450 4850 50  0001 C CNN
 	1    6450 4850
@@
 F 0 "R12" H 6720 4496 50  0000 L CNN
 F 1 "R" H 6720 4405 50  0000 L CNN
-F 2 "Resistor_THT:R_Axial_DIN0309_L9.0mm_D3.2mm_P12.70mm_Horizontal" V 6580 4450 50  0001 C CNN
+F 2 "Resistor_SMD:R_1206_3216Metric_Pad1.42x1.75mm_HandSolder" V 6580 4450 50  0001 C CNN
 F 3 "~" H 6650 4450 50  0001 C CNN
 	1    6650 4450
@@
 F 0 "R13" H 6970 4096 50  0000 L CNN
 F 1 "R" H 6970 4005 50  0000 L CNN
-F 2 "Resistor_THT:R_Axial_DIN0309_L9.0mm_D3.2mm_P12.70mm_Horizontal" V 6830 4050 50  0001 C CNN
+F 2 "Resistor_SMD:R_1206_3216Metric_Pad1.42x1.75mm_HandSolder" V 6830 4050 50  0001 C CNN
 F 3 "~" H 6900 4050 50  0001 C CNN
 	1    6900 4050

Commit message: Add chain guide models
Parts:
- added R14: R, Resistor_SMD:R_1206_3216Metric_Pad1.42x1.75mm_HandSolder, symbol Device:R
- D2, SW4: value MAN -> AUTO CTRL
- D3, SW3: value AP -> USR0
Connections:
- net +3V3: now also J1.1 (Pin_1), R14.2; no longer J1.2 (Pin_2)
- net GND: now also J1.2 (Pin_2); no longer J1.1 (Pin_1)
- net at R3.1: now also J1.6 (Pin_6); no longer J1.5 (Pin_5)
- net at R2.1: now also J1.5 (Pin_5); no longer J1.6 (Pin_6)
- net at J2.7 (Pin_7), R5.1: now also SW5.1; no longer SW3.1
- net at J2.5 (Pin_5): now also SW3.1, R14.1; no longer SW5.1
Other:
- moved on the sheet: D1, D2, D3, D5, D6, D7, R1, R2, R3, R7, R8, R9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
